File: kicad/nano-wallscout.kicad_sch (KiCad schematic)
At the start: 31 parts, among them Q1 IRLZ44N, SW1 Kalibrálás, SW2 Nullázás, U1 SSD1306, U2 MCP6004

Commit message: Add SVG diagram explaining flyback clipping: good vs bad scenarios
Parts:
- removed R12: 2k2, Resistor_THT:R_Axial_DIN0207_L6.3mm_D2.5mm_P10.16mm_Horizontal, symbol Device:R
- added R12: 2k2 heli, symbol Device:R_Trim
Connections:
- net at Lrx1.1, R11.1: now also R12.1
- net at Lrx1.2, R10.1, R7.1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: now also R12.2
Other:
- note added: "Az Ltx1 (Tx) és Lrx1 (RX) DD-ben átfedve: a közvetlen áthallás ≈ 0"
- note added: "Lecsengés csillapítás"
- note added: "OLED"
- note added: "Rx csillapítás"
- note added: "Soros védelem"
- note added: "Vbatt mérés"
- company: (none) -> BT-Soft
- title: (none) -> Arduino Nano betonvas kereső
Changed lines of the file:
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@@
 	(paper "A4")
 	(title_block
-		(date "sam. 04 avril 2015")
+		(title "Arduino Nano betonvas kereső")
+		(date "2026-10-25")
+		(rev "V1.0")
+		(company "BT-Soft")
 	)
 	(text "Vmid"
@@
 		)
 	)
+	(text "Az Ltx1 (Tx) és Lrx1 (RX) DD-ben átfedve: \na közvetlen áthallás ≈ 0"
+		(exclude_from_sim no)
+		(at 194.818 64.262 0)
+		(effects
+			(font
+				(size 1.27 1.27)
+			)
+		)
+	)
+	(text "Soros védelem"
+		(exclude_from_sim no)
+		(at 185.42 76.962 0)
+		(effects
+			(font
+				(size 1.27 1.27)
+			)
+		)
+	)
+	(text "Lecsengés\ncsillapítás"
+		(exclude_from_sim no)
+		(at 228.346 102.616 0)
+		(effects
+			(font
+				(size 1.27 1.27)
+			)
+		)
+	)
+	(text "OLED"
+		(exclude_from_sim no)
+		(at 47.752 139.954 0)
+		(effects
+			(font
+				(size 1.27 1.27)
+			)
+		)
+	)
+	(text "Vbatt mérés"
+		(exclude_from_sim no)
+		(at 85.09 67.564 0)
+		(effects
+			(font
+				(size 1.27 1.27)
+			)
+		)
+	)
+	(text "Rx csillapítás"
+		(exclude_from_sim no)
+		(at 186.944 108.966 90)
+		(effects
+			(font
+				(size 1.27 1.27)
+			)
+		)
+	)
 	(junction
 		(at 93.98 81.28)
@@
 	(symbol
 		(lib_id "Device:R")
-		(at 190.5 109.22 180)
-		(unit 1)
-		(body_style 1)
-		(exclude_from_sim no)
-		(in_bom yes)
-		(on_board yes)
-		(in_pos_files yes)
-		(dnp no)
-		(property "Reference" "R12"
-			(at 193.294 107.696 0)
-			(show_name no)
-			(do_not_autoplace no)
-			(effects
-				(font
-					(size 1.27 1.27)
-				)
-				(justify right)
-			)
-		)
-		(property "Value" "2k2"
-			(at 193.548 110.998 0)
-			(show_name no)
-			(do_not_autoplace no)
-			(effects
-				(font
-					(size 1.27 1.27)
-				)
-				(justify right)
-			)
-		)
-		(property "Footprint" "Resistor_THT:R_Axial_DIN0207_L6.3mm_D2.5mm_P10.16mm_Horizontal"
-			(at 192.278 109.22 90)
-			(hide yes)
-			(show_name no)
-			(do_not_autoplace no)
-			(effects
-				(font
-					(size 1.27 1.27)
-				)
-			)
-		)
-		(property "Datasheet" ""
-			(at 190.5 109.22 0)
-			(hide yes)
-			(show_name no)
-			(do_not_autoplace no)
-			(effects
-				(font
-					(size 1.27 1.27)
-				)
-			)
-		)
-		(property "Description" "Resistor"
-			(at 190.5 109.22 0)
-			(hide yes)
-			(show_name no)
-			(do_not_autoplace no)
-			(effects
-				(font
-					(size 1.27 1.27)
-				)
-			)
-		)
-		(pin "1"
-		)
-		(pin "2"
-		)
-		(instances
-			(project "nano-wallscout"
-				(path "/0d35483a-0b12-46cc-b9f2-896fd6831779"
-					(reference "R12")
-					(unit 1)
-				)
-			)
-		)
-	)
-	(symbol
-		(lib_id "Device:R")
 		(at 238.76 124.46 180)
 		(unit 1)
@@
 					(unit 1)
 				)
+			)
+		)
+	)
+	(symbol
+		(lib_id "Device:R_Trim")
+		(at 190.5 109.22 0)
+		(mirror y)
+		(unit 1)
+		(body_style 1)
+		(exclude_from_sim no)
+		(in_bom yes)
+		(on_board yes)
+		(in_pos_files yes)
+		(dnp no)
+		(fields_autoplaced yes)
+		(property "Reference" "R12"
+			(at 193.04 107.9499 0)
+			(show_name no)
+			(do_not_autoplace no)
+			(effects
+				(font
+					(size 1.27 1.27)
+				)
+				(justify right)
+			)
+		)
+		(property "Value" "2k2 heli"
+			(at 193.04 110.4899 0)
+			(show_name no)
+			(do_not_autoplace no)
+			(effects
+				(font
+					(size 1.27 1.27)
+				)
+				(justify right)
+			)
+		)
+		(property "Footprint" ""
+			(at 192.278 109.22 90)
+			(hide yes)
+			(show_name no)
+			(do_not_autoplace no)
+			(effects
+				(font
+					(size 1.27 1.27)
+				)
+			)
+		)
+		(property "Datasheet" ""
+			(at 190.5 109.22 0)
+			(hide yes)
+			(show_name no)
+			(do_not_autoplace no)
+			(effects
+				(font
+					(size 1.27 1.27)
+				)
+			)
+		)
+		(property "Description" "Trimmable resistor (preset resistor)"
+			(at 190.5 109.22 0)
+			(hide yes)
+			(show_name no)
+			(do_not_autoplace no)
+			(effects
+				(font
+					(size 1.27 1.27)
+				)
+			)
+		)
+		(pin "1"
+		)
+		(pin "2"
+		)
+		(instances
+			(project "nano-wallscout"
+				(path "/0d35483a-0b12-46cc-b9f2-896fd6831779"
+					(reference "R12")
+					(unit 1)
+				)

Commit message: Refactor config.h: Improve documentation and adjust constants
- Enhanced comments for clarity, breaking long lines into multiple lines for better readability.
- Increased the weight of the exponential smoothing in normal mode from 0.3 to 0.5.
Parts:
- added C5: 100nF, symbol Device:C
- added C6: 1000uF/16V, symbol Device:C_Polarized
- added D1: 1N4148, symbol Device:D
- added Q1: 2N2222, symbol Device:Q_NPN
- added R1: 150, Resistor_THT:R_Axial_DIN0207_L6.3mm_D2.5mm_P10.16mm_Horizontal, symbol Device:R
- added R2: 1k, Resistor_THT:R_Axial_DIN0207_L6.3mm_D2.5mm_P10.16mm_Horizontal, symbol Device:R
- renumbered D1 to D2, D2 to D3, Q1 to Q2, R8 to R10, R9 to R11, R10 to R12, R11 to R13, R12 to R14, R13 to R15, R14 to R16, R15 to R17, R16 to R18, R1 to R3, R2 to R4, R3 to R5, R4 to R6, R5 to R7, R6 to R8, R7 to R9
Connections:
- net +5V: now also C5.2, C6.1, R1.2
- net GND: now also C5.1, C6.2, Q1.E; no longer BZ1.2 (-)
- net at BZ1.1 (+): now also D1.1 (K), R1.1; no longer A1.14 (D11)
- new net: BZ1.2 (-), D1.2 (A), Q1.C
- new net: A1.14 (D11), R2.1
- new net: Q1.B, R2.2
Other:
- moved on the sheet: BZ1, U1
