File: kicad/nano-wallscout-Nano/nano-wallscout.kicad_sch (KiCad schematic)
At the start: 37 parts, among them Q1 2N2222, Q2 IRLZ44N, SW1 Kalibrálás, SW2 Nullázás, U1 SSD1306, U2 MCP6004

Commit message: Atmel328P version, Buzzer on PD3 pin
Parts:
- removed R14: 2k2 heli, symbol Device:R_Trim
- removed R16: 4k7 heli, symbol Device:R_Trim
- added C3: 100nF, Capacitor_THT:C_Rect_L7.2mm_W2.5mm_P5.00mm, symbol Device:C
- added R14: 1k, Resistor_THT:R_Axial_DIN0207_L6.3mm_D2.5mm_P10.16mm_Horizontal, symbol Device:R
- added RV1: 2k, Potentiometer_THT:Potentiometer_Bourns_3266Y_Vertical, symbol Device:R_Potentiometer_Trim
- added RV2: 5k, Potentiometer_THT:Potentiometer_Bourns_3266Y_Vertical, symbol Device:R_Potentiometer_Trim
- BZ1: footprint (none) -> Buzzer_Beeper:Buzzer_TDK_PS1240P02BT_D12.2mm_H6.5mm
- C1: footprint (none) -> Capacitor_THT:C_Radial_D6.3mm_H11.0mm_P2.50mm
- C2: footprint (none) -> Capacitor_THT:C_Rect_L7.2mm_W2.5mm_P5.00mm
- C4: renamed from C3; footprint (none) -> Capacitor_THT:C_Rect_L7.2mm_W2.5mm_P5.00mm
- C5: renamed from C4; footprint (none) -> Capacitor_THT:C_Radial_D6.3mm_H11.0mm_P2.50mm
- C6: renamed from C5; footprint (none) -> Capacitor_THT:C_Rect_L7.2mm_W2.5mm_P5.00mm
- C7: renamed from C6; footprint (none) -> Capacitor_THT:CP_Radial_D10.0mm_P5.00mm
- D1: footprint (none) -> Diode_THT:D_DO-35_SOD27_P10.16mm_Horizontal
- D2: footprint (none) -> Diode_THT:D_DO-41_SOD81_P12.70mm_Horizontal
- D3: footprint (none) -> Diode_THT:D_DO-35_SOD27_P12.70mm_Horizontal
- Lrx1, Ltx1: footprint (none) -> TerminalBlock_Phoenix:TerminalBlock_Phoenix_PT-1,5-2-5.0-H_1x02_P5.00mm_Horizontal
- Q2: renamed from Q1; footprint (none) -> Package_TO_SOT_THT:TO-92_Inline_Wide
- SW1, SW2: footprint (none) -> Button_Switch_THT:SW_PUSH_6mm_H8mm
- U1: footprint Display:ER_OLEDM0.91_1x-I2C -> Display:128x64OLED
- U2: footprint (none) -> Package_DIP:DIP-14_W7.62mm_LongPads
- renumbered Q2 to Q1, R15 to R16, R17 to R18, R18 to R19
Connections:
- net GND: now also Q2.3 (E), C3.1; no longer Q2.E
- net at BZ1.2 (-), D1.2 (A): now also Q2.1 (C); no longer Q2.C
- net at Lrx1.1, R13.1: now also R14.2
- net at Lrx1.2, R12.1, R9.1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: now also RV1.2, RV1.3
- net at D2.2 (A), Ltx1.2, Q1.2 (D): now also RV2.2, RV2.3
- net at C5.1, R6.1, R7.2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: now also C3.2
- net at R16.1: now also RV2.1
- net at R2.1: now also A1.6 (D3); no longer A1.14 (D11)
- net at R2.2: now also Q2.2 (B); no longer Q2.B
- new net: R14.1, RV1.1
Other:
- moved on the sheet: R13, U2A
