File: kicad/nano-wallscout-Atmega328P/nano-wallscout-Atmega328P.kicad_pcb (KiCad board)
At the start: 2 copper layers, 52 parts, among them J1 +9-12V INPUT, J2 AVR-ISP-6, Q1 2N2222, Q2 IRLZ44N, SW1 Kalibrálás, SW2 Nullázás, SW3 Reset, U1 ATmega328P-P, U2 LM7805_TO220, U3 SSD1306, U4 MCP6004, Y1 16MHz

Commit message: update
Parts:
- renumbered D2 to D1, D1 to D2, Q2 to Q1, Q1 to Q2
Connections:
- U1 pad 14: BUZZER -> unconnected-(U1-PB0-Pad14)
- U1 pad 5: unconnected-(U1-PD3-Pad5) -> BUZZER
Changed lines of the file:
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@@
 			(layers "*.Cu" "*.Mask")
 			(remove_unused_layers no)
-			(net "Net-(Q1-B)")
+			(net "Net-(Q2-B)")
 			(pintype "passive")
 		)
@@
 			(remove_unused_layers no)
 			(roundrect_rratio 0.096154)
-			(net "Net-(D2-A)")
+			(net "Net-(D1-A)")
 			(pinfunction "Pin_1_1")
 			(pintype "passive")
@@
 		(descr "Diode, DO-41_SOD81 series, Axial, Horizontal, pin pitch=10.16mm, length*diameter=5.2*2.7mm^2, https://www.diodes.com/assets/Package-Files/DO-41-Plastic.pdf")
 		(tags "Diode DO-41_SOD81 series Axial Horizontal pin pitch 10.16mm  length 5.2mm diameter 2.7mm")
-		(property "Reference" "D2"
+		(property "Reference" "D1"
 			(at 5.08 -2.47 0)
 			(layer "F.SilkS")
@@
 			(layers "*.Cu" "*.Mask")
 			(remove_unused_layers no)
-			(net "Net-(D2-A)")
+			(net "Net-(D1-A)")
 			(pinfunction "A_2")
 			(pintype "passive")
@@
 		(descr "TO-92 leads in-line, wide, drill 0.75mm (see NXP sot054_po.pdf)")
 		(tags "to-92 sc-43 sc-43a sot54 PA33 transistor")
-		(property "Reference" "Q1"
+		(property "Reference" "Q2"
 			(at 2.54 -3.56 0)
 			(layer "F.SilkS")
@@
 			(layers "*.Cu" "*.Mask")
 			(remove_unused_layers no)
-			(net "Net-(Q1-B)")
+			(net "Net-(Q2-B)")
 			(pinfunction "B_2")
 			(pintype "input")
@@
 			(layers "*.Cu" "*.Mask")
 			(remove_unused_layers no)
-			(net "unconnected-(U1-PD3-Pad5)")
+			(net "BUZZER")
 			(pinfunction "PD3_5")
-			(pintype "bidirectional+no_connect")
+			(pintype "bidirectional")
 		)
 		(pad "6" thru_hole circle
@@
 			(layers "*.Cu" "*.Mask")
 			(remove_unused_layers no)
-			(net "BUZZER")
+			(net "unconnected-(U1-PB0-Pad14)")
 			(pinfunction "PB0_14")
-			(pintype "bidirectional")
+			(pintype "bidirectional+no_connect")
 		)
 		(pad "15" thru_hole circle
@@
 			(layers "*.Cu" "*.Mask")
 			(remove_unused_layers no)
-			(net "Net-(Q2-G)")
+			(net "Net-(Q1-G)")
 			(pintype "passive")
 		)
@@
 		(descr "Diode, DO-35_SOD27 series, Axial, Horizontal, pin pitch=10.16mm, length*diameter=4*2mm^2, http://www.diodes.com/_files/packages/DO-35.pdf")
 		(tags "Diode DO-35_SOD27 series Axial Horizontal pin pitch 10.16mm  length 4mm diameter 2mm")
-		(property "Reference" "D1"
+		(property "Reference" "D2"
 			(at 5.08 -2.12 0)
 			(layer "F.SilkS")
@@
 			(layers "*.Cu" "*.Mask")
 			(remove_unused_layers no)
-			(net "Net-(Q2-G)")
+			(net "Net-(Q1-G)")
 			(pintype "passive")
 		)
@@
 		(descr "TO-220-3, Vertical, RM 2.54mm, see https://www.vishay.com/docs/66542/to-220-1.pdf")
 		(tags "TO-220-3 Vertical RM 2.54mm")
-		(property "Reference" "Q2"
+		(property "Reference" "Q1"
 			(at 2.54 -4.1 0)
 			(layer "F.SilkS")
@@
 			(layers "*.Cu" "*.Mask")
 			(remove_unused_layers no)
-			(net "Net-(Q2-G)")
+			(net "Net-(Q1-G)")
 			(pinfunction "G_1")
 			(pintype "input")

Commit message: Atmel328P version PCB update
Parts:
- added TP2: Vétel beállítás, TestPoint:TestPoint_Loop_D2.50mm_Drill1.0mm, F.Cu at (96.8, 59.2)
- C10, C12, C2: footprint Capacitor_THT:C_Radial_D6.3mm_H11.0mm_P2.50mm -> Capacitor_THT:CP_Radial_D6.3mm_P2.50mm
- Lrx1, Ltx1: footprint TerminalBlock_Phoenix:TerminalBlock_Phoenix_PT-1,5-2-5.0-H_1x02_P5.00mm_Horizontal -> TerminalBlock_Phoenix:TerminalBlock_Phoenix_PT-1,5-3-3.5-H_1x03_P3.50mm_Horizontal
- U2: value LM7805_TO220 -> LM7805
- U3: footprint Display:128x64OLED -> Connector_PinHeader_2.54mm:PinHeader_1x04_P2.54mm_Vertical
- moved C10 111.8 mm to (70.8, 30.8), turned to 90 degrees
- moved U2 104.6 mm to (72.0, 62.2)
- moved RV2 102.7 mm to (100.0, 27.2), turned to 180 degrees
- moved C8 94.6 mm to (71.0, 34.5), turned to -90 degrees
- moved C9 93.4 mm to (85.2, 26.0)
- moved RV1 93.4 mm to (101.2, 31.2), turned to 90 degrees
- moved C2 92.1 mm to (73.5, 69.0), turned to 90 degrees
- moved C5 92.0 mm to (76.5, 48.0), turned to 180 degrees
- moved D3 87.7 mm to (119.0, 46.8), turned to 90 degrees
- moved U4 84.4 mm to (92.8, 48.9), turned to 180 degrees
- moved R18 83.9 mm to (106.8, 38.8), turned to -90 degrees
- moved R17 83.2 mm to (122.2, 36.7), turned to -90 degrees
- moved C4 80.2 mm to (71.8, 56.0)
- moved R16 79.9 mm to (125.8, 36.7), turned to -90 degrees
- moved Ltx1 79.5 mm to (127.5, 28.6), turned to 180 degrees
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Connections:
- R3 pad 1: Net-(U1-~{RESET}/PC6) -> /RESET
- SW3 pad 2: Net-(U1-~{RESET}/PC6) -> /RESET
- U1 pad 1: Net-(U1-~{RESET}/PC6) -> /RESET
Routing:
- net GND: track 0.00 -> 445.2 mm
- net +5V: track 0.00 -> 174.1 mm
- net +BATT: track 0.00 -> 105.2 mm
- net Net-(U4C--): track 0.00 -> 67.1 mm
- net /RESET: track 0.00 -> 59.8 mm
- net D2/Tx: track 0.00 -> 57.7 mm
- net Net-(D3-A): track 0.00 -> 40.8 mm
- net Net-(U4D-+): track 0.00 -> 36.5 mm
- net Net-(Lrx1-Pad1): track 0.00 -> 34.4 mm
- net Zero: track 0.00 -> 30.9 mm
- net Calib: track 0.00 -> 28.5 mm
- net Net-(U4C-+): track 0.00 -> 24.4 mm
- net Net-(Q1-G): track 0.00 -> 21.9 mm
- net OLED SCL: track 0.00 -> 21.5 mm
- net OLED SDA: track 0.00 -> 20.6 mm
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Other:
- board outline added: 63.8 x 75 mm
- board text added: "BT-Soft 2026"
- board text added: "Nano WallScout"
