File: kicad/nano-wallscout-Atmega328P/nano-wallscout-Atmega328P.kicad_pcb (KiCad board)
At the start: 2 copper layers, 63.8 x 75 mm, 53 parts, among them J1 +9-12V INPUT, J2 AVR-ISP-6, Q1 IRLZ44N, Q2 2N2222, SW1 Kalibrálás, SW2 Nullázás, SW3 Reset, U1 ATmega328P-P, U2 LM7805, U3 SSD1306, U4 MCP6004, Y1 16MHz

Commit message: update
Parts:
- moved J2 0.92 mm to (126.0, 72.1)
Routing:
- net GND: track 445.2 -> 441.2 mm
- net Net-(Q1-G): track 21.9 -> 23.0 mm
- net MOSI: track 15.0 -> 15.9 mm
- net SCK: track 17.6 -> 18.5 mm
- net +5V: track 174.1 -> 174.9 mm
- net Net-(U4A--): track 16.9 -> 17.6 mm
- net MISO: track 15.7 -> 16.4 mm
Other:
- board text added: "Nano WallScout BT-Soft 2026"
- board text removed: "Nano WallScout"

Commit message: update
Parts:
- renumbered D2 to D1, D3 to D2, D4 to D3, D1 to D4
Changed lines of the file:
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@@
 			(layers "*.Cu" "*.Mask")
 			(remove_unused_layers no)
-			(net "Net-(D3-A)")
+			(net "Net-(D2-A)")
 			(pinfunction "2_2")
 			(pintype "passive")
@@
 			(remove_unused_layers no)
 			(roundrect_rratio 0.096154)
-			(net "Net-(D1-A)")
+			(net "Net-(D4-A)")
 			(pinfunction "Pin_1_1")
 			(pintype "passive")
@@
 		(descr "Diode, DO-41_SOD81 series, Axial, Horizontal, pin pitch=10.16mm, length*diameter=5.2*2.7mm^2, https://www.diodes.com/assets/Package-Files/DO-41-Plastic.pdf")
 		(tags "Diode DO-41_SOD81 series Axial Horizontal pin pitch 10.16mm  length 5.2mm diameter 2.7mm")
-		(property "Reference" "D1"
+		(property "Reference" "D4"
 			(at 5.08 -2.47 90)
 			(layer "F.SilkS")
@@
 			(layers "*.Cu" "*.Mask")
 			(remove_unused_layers no)
-			(net "Net-(D1-A)")
+			(net "Net-(D4-A)")
 			(pinfunction "A_2")
 			(pintype "passive")
@@
 		(descr "Diode, DO-35_SOD27 series, Axial, Horizontal, pin pitch=10.16mm, length*diameter=4*2mm^2, http://www.diodes.com/_files/packages/DO-35.pdf")
 		(tags "Diode DO-35_SOD27 series Axial Horizontal pin pitch 10.16mm  length 4mm diameter 2mm")
-		(property "Reference" "D4"
+		(property "Reference" "D3"
 			(at 5.08 -2.12 90)
 			(layer "F.SilkS")
@@
 			(remove_unused_layers no)
 			(roundrect_rratio 0.15625)
-			(net "Net-(D3-K)")
+			(net "Net-(D2-K)")
 			(pinfunction "K_1")
 			(pintype "passive")
@@
 		(descr "Diode, DO-35_SOD27 series, Axial, Horizontal, pin pitch=10.16mm, length*diameter=4*2mm^2, http://www.diodes.com/_files/packages/DO-35.pdf")
 		(tags "Diode DO-35_SOD27 series Axial Horizontal pin pitch 10.16mm  length 4mm diameter 2mm")
-		(property "Reference" "D3"
+		(property "Reference" "D2"
 			(at 5.08 -2.12 90)
 			(layer "F.SilkS")
@@
 			(remove_unused_layers no)
 			(roundrect_rratio 0.15625)
-			(net "Net-(D3-K)")
+			(net "Net-(D2-K)")
 			(pinfunction "K_1")
 			(pintype "passive")
@@
 			(layers "*.Cu" "*.Mask")
 			(remove_unused_layers no)
-			(net "Net-(D3-A)")
+			(net "Net-(D2-A)")
 			(pinfunction "A_2")
 			(pintype "passive")
@@
 			(layers "*.Cu" "*.Mask")
 			(remove_unused_layers no)
-			(net "Net-(D3-A)")
+			(net "Net-(D2-A)")
 			(pinfunction "2_2")
 			(pintype "passive")
@@
 			(layers "*.Cu" "*.Mask")
 			(remove_unused_layers no)
-			(net "Net-(D3-A)")
+			(net "Net-(D2-A)")
 			(pinfunction "3_3")
 			(pintype "passive")
@@
 			)
 		)
-		(property "Description" "SSD1306 OLED module, 0.91 inch, 128x32, I2C"
+		(property "Description" "SSD1306 OLED module, 0.91 inch, 128x64, I2C"
 			(at 0 0 90)
 			(layer "F.Fab")
@@
 		(descr "Diode, DO-35_SOD27 series, Axial, Horizontal, pin pitch=10.16mm, length*diameter=4*2mm^2, http://www.diodes.com/_files/packages/DO-35.pdf")
 		(tags "Diode DO-35_SOD27 series Axial Horizontal pin pitch 10.16mm  length 4mm diameter 2mm")
-		(property "Reference" "D2"
+		(property "Reference" "D1"
 			(at 5.08 -2.12 90)
 			(layer "F.SilkS")
@@
 			(layers "*.Cu" "*.Mask")
 			(remove_unused_layers no)
-			(net "Net-(D3-A)")
+			(net "Net-(D2-A)")
 			(pinfunction "D_2")
 			(pintype "passive")
@@
 	)
 	(segment
-		(start 116.96 40.79)
-		(end 119 38.75)
-		(width 0.8)
-		(layer "B.Cu")
-		(net "Net-(D3-A)")
-	)
-	(segment
-		(start 119 36.59)
-		(end 119 35.25)
-		(width 0.8)
-		(layer "B.Cu")
-		(net "Net-(D3-A)")
-	)
-	(segment
-		(start 105.08 30.58)
-		(end 108.75 34.25)
-		(width 0.2)
-		(layer "B.Cu")
-		(net "Net-(D3-A)")
-	)
-	(segment
-		(start 123.25 32.25)
-		(end 124 31.5)
-		(width 0.8)
-		(layer "B.Cu")
-		(net "Net-(D3-A)")
-	)
-	(segment
-		(start 110.29 40.79)
-		(end 112 40.79)
-		(width 0.2)
-		(layer "B.Cu")
-		(net "Net-(D3-A)")
-	)
-	(segment
-		(start 108.75 39.25)
-		(end 110.29 40.79)
-		(width 0.2)
-		(layer "B.Cu")
-		(net "Net-(D3-A)")
-	)
-	(segment
-		(start 119 38.75)
-		(end 119 36.59)
-		(width 0.8)
-		(layer "B.Cu")
-		(net "Net-(D3-A)")
-	)
-	(segment
-		(start 105.08 27.25)
-		(end 105.08 30.58)
-		(width 0.2)
-		(layer "B.Cu")
-		(net "Net-(D3-A)")
-	)
-	(segment
-		(start 108.75 34.25)
-		(end 108.75 39.25)
-		(width 0.2)
-		(layer "B.Cu")
-		(net "Net-(D3-A)")
-	)
-	(segment
-		(start 119 35.25)
-		(end 122 32.25)
-		(width 0.8)
-		(layer "B.Cu")
-		(net "Net-(D3-A)")
-	)
-	(segment
-		(start 102.54 27.25)
-		(end 105.08 27.25)
-		(width 0.2)
-		(layer "B.Cu")
-		(net "Net-(D3-A)")
-	)
-	(segment
-		(start 112 40.79)
-		(end 116.96 40.79)
-		(width 0.8)
-		(layer "B.Cu")
-		(net "Net-(D3-A)")
-	)
-	(segment
-		(start 122 32.25)
-		(end 123.25 32.25)
-		(width 0.8)
-		(layer "B.Cu")
-		(net "Net-(D3-A)")
-	)
-	(segment
-		(start 124 31.5)
-		(end 124 28.5825)
-		(width 0.8)
-		(layer "B.Cu")
-		(net "Net-(D3-A)")
-	)
-	(segment
 		(start 100.29 63.87)
 		(end 99.13 63.87)
@@
 	)
 	(segment
-		(start 73.5 83.33)
-		(end 73.5 88.5)
-		(width 0.2)
-		(layer "B.Cu")
-		(net "Net-(D1-A)")
-	)
-	(segment
 		(start 90 41.25)
 		(end 92.81 41.25)
@@
 	)
 	(segment
-		(start 116.25 46.75)
-		(end 119 46.75)
-		(width 0.2)
-		(layer "B.Cu")
-		(net "Net-(D3-K)")
-	)
-	(segment
 		(start 124.5 80.75)
 		(end 126.25 82.5)
@@
 		(net "Net-(Q1-G)")
 	)
+	(segment
+		(start 116.96 40.79)
+		(end 119 38.75)
+		(width 0.8)
+		(layer "B.Cu")
+		(net "Net-(D2-A)")
+	)
+	(segment
+		(start 119 36.59)
+		(end 119 35.25)
+		(width 0.8)
+		(layer "B.Cu")
+		(net "Net-(D2-A)")
+	)
+	(segment
+		(start 105.08 30.58)
+		(end 108.75 34.25)
+		(width 0.2)
+		(layer "B.Cu")
+		(net "Net-(D2-A)")
+	)
+	(segment
+		(start 123.25 32.25)
+		(end 124 31.5)
+		(width 0.8)
+		(layer "B.Cu")
+		(net "Net-(D2-A)")
+	)
+	(segment
+		(start 110.29 40.79)
+		(end 112 40.79)
+		(width 0.2)
+		(layer "B.Cu")
+		(net "Net-(D2-A)")
+	)
+	(segment
+		(start 108.75 39.25)
+		(end 110.29 40.79)
+		(width 0.2)
+		(layer "B.Cu")
+		(net "Net-(D2-A)")
+	)
+	(segment
+		(start 119 38.75)
+		(end 119 36.59)
+		(width 0.8)
+		(layer "B.Cu")
+		(net "Net-(D2-A)")
+	)
+	(segment
+		(start 105.08 27.25)
+		(end 105.08 30.58)
+		(width 0.2)
+		(layer "B.Cu")
+		(net "Net-(D2-A)")
+	)
+	(segment
+		(start 108.75 34.25)
+		(end 108.75 39.25)
+		(width 0.2)
+		(layer "B.Cu")
+		(net "Net-(D2-A)")
+	)
+	(segment
+		(start 119 35.25)
+		(end 122 32.25)
+		(width 0.8)
+		(layer "B.Cu")
+		(net "Net-(D2-A)")
+	)
+	(segment
+		(start 102.54 27.25)
+		(end 105.08 27.25)
+		(width 0.2)
+		(layer "B.Cu")
+		(net "Net-(D2-A)")
+	)
+	(segment
+		(start 112 40.79)
+		(end 116.96 40.79)
+		(width 0.8)
+		(layer "B.Cu")
+		(net "Net-(D2-A)")
+	)
+	(segment
+		(start 122 32.25)
+		(end 123.25 32.25)
+		(width 0.8)
+		(layer "B.Cu")
+		(net "Net-(D2-A)")
+	)
+	(segment
+		(start 124 31.5)
+		(end 124 28.5825)
+		(width 0.8)
+		(layer "B.Cu")
+		(net "Net-(D2-A)")
+	)
+	(segment
+		(start 116.25 46.75)
+		(end 119 46.75)
+		(width 0.2)
+		(layer "B.Cu")
+		(net "Net-(D2-K)")
+	)
+	(segment
+		(start 73.5 83.33)
+		(end 73.5 88.5)
+		(width 0.2)
+		(layer "B.Cu")
+		(net "Net-(D4-A)")
+	)
 	(embedded_fonts no)
