File: kicad/nano-wallscout-Atmega328P/nano-wallscout-Atmega328P.kicad_sch (KiCad schematic)
At the start: 52 parts, among them J1 +9-12V INPUT, J2 AVR-ISP-6, Q1 IRLZ44N, Q2 2N2222, SW1 Kalibrálás, SW2 Nullázás, SW3 Reset, U1 ATmega328P-P, U2 LM7805_TO220, U3 SSD1306, U4 MCP6004, Y1 16MHz

Commit message: Atmel328P version PCB update
Parts:
- removed Lrx1, Ltx1: 1mH, TerminalBlock_Phoenix:TerminalBlock_Phoenix_PT-1,5-2-5.0-H_1x02_P5.00mm_Horizontal, symbol Device:L
- added Lrx1, Ltx1: 1mH, TerminalBlock_Phoenix:TerminalBlock_Phoenix_PT-1,5-3-3.5-H_1x03_P3.50mm_Horizontal, symbol WallScout-Kicad-library:L-Shield
- added TP2: Vétel beállítás, TestPoint:TestPoint_Loop_D2.50mm_Drill1.0mm, symbol Connector:TestPoint_Alt
- C10, C12, C2: footprint Capacitor_THT:C_Radial_D6.3mm_H11.0mm_P2.50mm -> Capacitor_THT:CP_Radial_D6.3mm_P2.50mm
- U2: value LM7805_TO220 -> LM7805
- U3: footprint Display:128x64OLED -> Connector_PinHeader_2.54mm:PinHeader_1x04_P2.54mm_Vertical
Connections:
- net +BATT: now also Ltx1.1
- net A0/Rx: now also TP2.1
- net GND: now also Lrx1.3 (SHIELD), Ltx1.3 (SHIELD)
- net /RESET: now also R3.1, SW3.2, U1.1 (~{RESET}/PC6)
- net at R13.1, R8.1, RV1.2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: now also Lrx1.2
- net at D3.2 (A), Q1.2 (D), RV2.2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: now also Ltx1.2
- net at R14.1, R15.2: now also Lrx1.1
Other:
- note added: "Árnyékolt tekercsek"
- note removed: "Reset"
