File: kicad/nano-wallscout-Atmega328P/nano-wallscout-Atmega328P.kicad_sch (KiCad schematic)
At the start: 53 parts, among them J1 +9-12V INPUT, J2 AVR-ISP-6, Q1 IRLZ44N, Q2 2N2222, SW1 Kalibrálás, SW2 Nullázás, SW3 Reset, U1 ATmega328P-P, U2 LM7805, U3 SSD1306, U4 MCP6004, Y1 16MHz

Commit message: update
Parts:
- renumbered D2 to D1, D3 to D2, D4 to D3, D1 to D4, U4 to U2, U2 to U4
Changed lines of the file:
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@@
 		(in_pos_files yes)
 		(dnp no)
-		(property "Reference" "D3"
+		(property "Reference" "D2"
 			(at 269.24 129.5399 90)
 			(show_name no)
@@
 			(project "nano-wallscout-Atmega328P"
 				(path "/34d29903-802b-4e4f-a971-54513bc11f78"
-					(reference "D3")
+					(reference "D2")
 					(unit 1)
 				)
@@
 		(in_pos_files yes)
 		(dnp no)
-		(property "Reference" "U4"
+		(property "Reference" "U2"
 			(at 168.656 107.442 0)
 			(show_name no)
@@
 			(project "nano-wallscout-Atmega328P"
 				(path "/34d29903-802b-4e4f-a971-54513bc11f78"
-					(reference "U4")
+					(reference "U2")
 					(unit 3)
 				)
@@
 		(dnp no)
 		(fields_autoplaced yes)
-		(property "Reference" "D2"
+		(property "Reference" "D1"
 			(at 43.18 162.5599 90)
 			(show_name no)
@@
 			(project "nano-wallscout-Atmega328P"
 				(path "/34d29903-802b-4e4f-a971-54513bc11f78"
-					(reference "D2")
+					(reference "D1")
 					(unit 1)
 				)
@@
 		(dnp no)
 		(fields_autoplaced yes)
-		(property "Reference" "D1"
+		(property "Reference" "D4"
 			(at 40.64 24.13 0)
 			(show_name no)
@@
 			(project "nano-wallscout-Atmega328P"
 				(path "/34d29903-802b-4e4f-a971-54513bc11f78"
-					(reference "D1")
+					(reference "D4")
 					(unit 1)
 				)
@@
 		(dnp no)
 		(fields_autoplaced yes)
-		(property "Reference" "U2"
+		(property "Reference" "U4"
 			(at 72.39 24.13 0)
 			(show_name no)
@@
 			(project "nano-wallscout-Atmega328P"
 				(path "/34d29903-802b-4e4f-a971-54513bc11f78"
-					(reference "U2")
+					(reference "U4")
 					(unit 1)
 				)
@@
 		(in_pos_files yes)
 		(dnp no)
-		(property "Reference" "U4"
+		(property "Reference" "U2"
 			(at 174.752 70.104 0)
 			(show_name no)
@@
 			(project "nano-wallscout-Atmega328P"
 				(path "/34d29903-802b-4e4f-a971-54513bc11f78"
-					(reference "U4")
+					(reference "U2")
 					(unit 2)
 				)
@@
 		(in_pos_files yes)
 		(dnp no)
-		(property "Reference" "U4"
+		(property "Reference" "U2"
 			(at 206.248 66.802 0)
 			(show_name no)
@@
 			(project "nano-wallscout-Atmega328P"
 				(path "/34d29903-802b-4e4f-a971-54513bc11f78"
-					(reference "U4")
+					(reference "U2")
 					(unit 1)
 				)
@@
 		(in_pos_files yes)
 		(dnp no)
-		(property "Reference" "U4"
+		(property "Reference" "U2"
 			(at 151.892 72.39 0)
 			(show_name no)
@@
 			(project "nano-wallscout-Atmega328P"
 				(path "/34d29903-802b-4e4f-a971-54513bc11f78"
-					(reference "U4")
+					(reference "U2")
 					(unit 4)
 				)
@@
 		(in_pos_files yes)
 		(dnp no)
-		(property "Reference" "D4"
+		(property "Reference" "D3"
 			(at 269.24 140.9699 90)
 			(show_name no)
@@
 			(project "nano-wallscout-Atmega328P"
 				(path "/34d29903-802b-4e4f-a971-54513bc11f78"
-					(reference "D4")
+					(reference "D3")
 					(unit 1)
 				)
@@
 		(dnp no)
 		(property "Reference" "R16"
-			(at 228.854 141.478 90)
+			(at 228.6 133.35 90)
 			(show_name no)
 			(do_not_autoplace no)
@@
 		)
 		(property "Value" "100"
-			(at 229.108 138.938 90)
+			(at 228.854 138.684 90)
 			(show_name no)
 			(do_not_autoplace no)

Commit message: update
Parts:
- renumbered Q2 to Q1, Q1 to Q2
Changed lines of the file:
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@@
 		(in_pos_files yes)
 		(dnp no)
-		(property "Reference" "Q1"
+		(property "Reference" "Q2"
 			(at 248.412 125.73 0)
 			(show_name no)
@@
 			(project "nano-wallscout-Atmega328P"
 				(path "/34d29903-802b-4e4f-a971-54513bc11f78"
-					(reference "Q1")
+					(reference "Q2")
 					(unit 1)
 				)
@@
 		(dnp no)
 		(fields_autoplaced yes)
-		(property "Reference" "Q2"
+		(property "Reference" "Q1"
 			(at 34.29 177.7999 0)
 			(show_name no)
@@
 			(project "nano-wallscout-Atmega328P"
 				(path "/34d29903-802b-4e4f-a971-54513bc11f78"
-					(reference "Q2")
-					(unit 1)
-				)
+					(reference "Q1")
+					(unit 1)
+				)

Commit message: HandHeld harware SCH+PCB begin
Parts:
- renumbered U4 to U2
Changed lines of the file:
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@@
 		(dnp no)
 		(fields_autoplaced yes)
-		(property "Reference" "U4"
-			(at 153.67 171.4499 0)
+		(property "Reference" "U2"
+			(at 156.21 171.4499 0)
 			(show_name no)
 			(do_not_autoplace no)
@@
 					(size 1.27 1.27)
 				)
-				(justify left)
+				(justify right)
 			)
 		)
 		(property "Value" "MCP6004"
-			(at 153.67 173.9899 0)
+			(at 156.21 173.9899 0)
 			(show_name no)
 			(do_not_autoplace no)
@@
 					(size 1.27 1.27)
 				)
-				(justify left)
+				(justify right)
 			)
 		)
@@
 			(project "nano-wallscout-Atmega328P"
 				(path "/34d29903-802b-4e4f-a971-54513bc11f78"
-					(reference "U4")
+					(reference "U2")
 					(unit 5)
 				)
